Commit message: isaac setting

File: fanuc_hardware_interface/config/crx_mock_ros2_control_macro.xacro (robot description, xacro)
@@ -1,5 +1,10 @@
 <?xml version="1.0"?>
 <robot xmlns:xacro="http://wiki.ros.org/xacro">
-  <xacro:macro name="crx_control" params="name prefix=''">
+  <xacro:macro name="crx_control" params="
+    name
+    prefix=''
+    sim_isaac=false
+    mock_sensor_commands=false
+    gripper_closed_position=0.7929">
     <ros2_control name="${name}" type="system">
       <joint name="${prefix}J1">
@@ -30,4 +35,34 @@
       <joint name="${prefix}J6">
         <command_interface name="position"/>
+        <state_interface name="position"/>
+        <state_interface name="velocity"/>
+      </joint>
+      <!-- gripper -->
+      <!-- Joint interfaces -->
+      <!-- With Gazebo or Hardware, they handle mimic joints, so we only need this command interface activated -->
+      <joint name="${prefix}finger_joint">
+        <command_interface name="position" />
+        <state_interface name="position">
+          <param name="initial_value">${gripper_closed_position}</param>
+        </state_interface>
+        <state_interface name="velocity"/>
+      </joint>
+      <joint name="${prefix}right_outer_knuckle_joint">
+        <state_interface name="position"/>
+        <state_interface name="velocity"/>
+      </joint>
+      <joint name="${prefix}left_inner_finger_knuckle_joint">
+        <state_interface name="position"/>
+        <state_interface name="velocity"/>
+      </joint>
+      <joint name="${prefix}right_inner_finger_knuckle_joint">
+        <state_interface name="position"/>
+        <state_interface name="velocity"/>
+      </joint>
+      <joint name="${prefix}left_inner_finger_joint">
+        <state_interface name="position"/>
+        <state_interface name="velocity"/>
+      </joint>
+      <joint name="${prefix}right_inner_finger_joint">
         <state_interface name="position"/>
         <state_interface name="velocity"/>
@@ -172,4 +207,8 @@
         <state_interface name="tp_enabled"/>
       </gpio>
+      <gpio name="reactivate_gripper">
+        <command_interface name="reactivate_gripper_cmd" />
+        <command_interface name="reactivate_gripper_response" />
+      </gpio>
       <sensor name="Force">
         <state_interface name="force_x"/>
@@ -193,4 +232,6 @@
         <param name="state_following_offset">0.0</param>
         <param name="calculate_dynamics">true</param>
+        <param name="mock_sensor_commands">${mock_sensor_commands}</param>
+        <param name="state_following_offset">0.0</param>
       </hardware>
     </ros2_control>

File: fanuc_hardware_interface/config/crx_physical_ros2_control_macro.xacro (robot description, xacro)
@@ -1,5 +1,15 @@
 <?xml version="1.0"?>
 <robot xmlns:xacro="http://wiki.ros.org/xacro">
-  <xacro:macro name="crx_control" params="name prefix=''">
+  <xacro:macro name="crx_control" params="
+    name
+    prefix=''
+    sim_isaac=false
+    mock_sensor_commands:=false
+    com_port:=/dev/ttyUSB0
+    gripper_speed_multiplier:=1.0
+    gripper_force_multiplier:=0.5
+    gripper_max_speed:=0.150
+    gripper_max_force:=235.0
+    gripper_closed_position:=0.7929">
     <ros2_control name="${name}" type="system">
       <joint name="${prefix}J1">
@@ -33,14 +43,37 @@
         <state_interface name="velocity"/>
       </joint>
+      <!-- gripper -->
+      <!-- Joint interfaces -->
+      <!-- With Gazebo or Hardware, they handle mimic joints, so we only need this command interface activated -->
+      <joint name="${prefix}finger_joint">
+        <command_interface name="position"/>
+        <state_interface name="position"/>
+        <state_interface name="velocity"/>
+      </joint>
       <hardware>
-        <plugin>fanuc_robot_driver/FanucHardwareInterface</plugin>
-        <param name="robot_ip">$(arg robot_ip)</param>
-        <param name="rmi_port">$(arg rmi_port)</param>
-        <param name="stream_motion_port">$(arg stream_motion_port)</param>
-        <param name="gpio_configuration">$(arg gpio_configuration)</param>
-        <param name="payload_schedule">$(arg payload_schedule)</param>
-        <param name="out_cmd_interp_buff_target">$(arg out_cmd_interp_buff_target)</param>
-        <param name="force_sensor_type">$(arg force_sensor_type)</param>
-	<param name="motion_control">$(arg motion_control)</param>
+        <xacro:if value="${sim_isaac}">
+          <plugin>topic_based_ros2_control/TopicBasedSystem</plugin>
+          <param name="joint_commands_topic">isaac_joint_commands</param>
+          <param name="joint_states_topic">isaac_joint_states</param>
+          <param name="trigger_joint_command_threshold">0.02</param>
+        </xacro:if>
+        <xacro:unless value="${sim_isaac}">
+          <plugin>fanuc_robot_driver/FanucHardwareInterface</plugin>
+          <plugin>robotiq_driver/RobotiqGripperHardwareInterface</plugin>
+          <param name="robot_ip">$(arg robot_ip)</param>
+          <param name="rmi_port">$(arg rmi_port)</param>
+          <param name="stream_motion_port">$(arg stream_motion_port)</param>
+          <param name="gpio_configuration">$(arg gpio_configuration)</param>
+          <param name="payload_schedule">$(arg payload_schedule)</param>
+          <param name="out_cmd_interp_buff_target">$(arg out_cmd_interp_buff_target)</param>
+          <param name="force_sensor_type">$(arg force_sensor_type)</param>
+          <param name="motion_control">$(arg motion_control)</param>
+          <param name="gripper_closed_position">${gripper_closed_position}</param>
+          <param name="COM_port">${com_port}</param>
+          <param name="gripper_speed_multiplier">${gripper_speed_multiplier}</param>
+          <param name="gripper_force_multiplier">${gripper_force_multiplier}</param>
+          <param name="gripper_max_speed">${gripper_max_speed}</param>
+          <param name="gripper_max_force">${gripper_max_force}</param>
+        </xacro:unless>
       </hardware>
     </ros2_control>

File: fanuc_hardware_interface/robot/crx5ia_2f_85gripper.urdf.xacro (robot description, xacro)
@@ -9,4 +9,5 @@
   <xacro:arg name="force_sensor_type" default="1"/>
   <xacro:arg name="use_mock" default="false"/>
+  <xacro:arg name="sim_isaac" default="false"/>
   <xacro:arg name="motion_control" default="1"/>
   <xacro:arg name="origin_xyz" default="0 0 0"/>
@@ -18,4 +19,9 @@
   <xacro:arg name="use_fake_hardware" default="true" />
   <xacro:arg name="com_port" default="/dev/ttyUSB0" />
+  <xacro:arg name="gripper_closed_position" default="0.7929" />
+  <xacro:arg name="gripper_speed_multiplier" default="1.0" />
+  <xacro:arg name="gripper_force_multiplier" default="0.5" />
+  <xacro:arg name="gripper_max_speed" default="0.150" />
+  <xacro:arg name="gripper_max_force" default="235.0" />
   <xacro:include filename="$(find fanuc_crx_description)/urdf/crx5ia_2f_85gripper_urdf_macro.xacro"/>
   <xacro:if value="$(arg use_mock)">
@@ -30,4 +36,4 @@
     <origin xyz="$(arg origin_xyz)" rpy="$(arg origin_rpy)"/>
   </xacro:crx5ia_2f_85gripper>
-  <xacro:crx_control name="crx5ia_2f_85gripper" prefix="$(arg prefix)"/>
+  <xacro:crx_control name="crx5ia_2f_85gripper" prefix="$(arg prefix)" sim_isaac="$(arg sim_isaac)"/>
 </robot>
